Commit message: message

File: src/mp_description/urdf/mp.urdf.xacro (robot description, xacro)
@@ -113,8 +113,7 @@
         </visual>
         <collision>
-            <origin rpy="${PI/2} 0 0" xyz="-0.4 0.4 0"/>
-            <geometry>
-                <mesh filename="package://mp_description/meshes/mp_link1.STL" scale= "0.01 0.01 0.01"/>
-                <!-- changed link1, link2, link3, link4 collision scaled to 0.01-->
+            <origin rpy="${PI} ${PI/2} ${PI}" xyz="-0.4 0.4 0"/>
+            <geometry>
+                <cylinder radius="0.1" length="0.1"/> <!-- Adjust dimensions -->
             </geometry>
         </collision>
@@ -135,7 +134,7 @@
         </visual>
         <collision>
-            <origin rpy="${PI} 0 ${PI}" xyz="0.3 -0.3 1"/>
-            <geometry>
-                <mesh filename="package://mp_description/meshes/mp_link2.STL" scale= "0.01 0.01 0.01"/>
+            <origin rpy="${PI} ${PI/2} ${PI}" xyz="0.3 -0.3 1"/>
+            <geometry>
+                <cylinder radius="0.1" length="0.1"/> <!-- Adjust dimensions -->
             </geometry>
         </collision>
@@ -157,7 +156,7 @@
         </visual>
         <collision>
-            <origin rpy="0 -${PI/2} 0" xyz="0.4 -0.25 0.0"/>
-            <geometry>
-                <mesh filename="package://mp_description/meshes/mp_link3.STL" scale= "0.01 0.01 0.01"/>
+            <origin rpy="${PI} ${PI/2} ${PI}" xyz="0.4 -0.25 0.0"/>
+            <geometry>
+                <cylinder radius="0.1" length="0.1"/> <!-- Adjust dimensions -->
             </geometry>
         </collision>
@@ -179,7 +178,7 @@
         </visual>
         <collision>
-            <origin rpy="0 -${PI/2} 0" xyz="0.4 -0.25 -0.65"/>
-            <geometry>
-                <mesh filename="package://mp_description/meshes/mp_link4.STL" scale= "0.01 0.01 0.01"/>
+            <origin rpy="${PI} ${PI/2} ${PI}" xyz="0.4 -0.25 -0.65"/>
+            <geometry>
+                <cylinder radius="0.1" length="0.1"/> <!-- Adjust dimensions -->
             </geometry>
         </collision>
@@ -203,5 +202,5 @@
             <origin rpy="${PI} ${PI/2} ${PI}" xyz="-0.3 -0.2 0.6"/>
             <geometry>
-                <mesh filename="package://mp_description/meshes/mp_link5.STL" scale= "0.01 0.01 0.01"/>
+                <cylinder radius="0.1" length="0.1"/> <!-- Adjust dimensions -->
             </geometry>
         </collision>
@@ -223,7 +222,7 @@
         </visual>
         <collision>
-            <origin rpy="${PI/2} 0 0" xyz="-0.25 0.25 0"/>
-            <geometry>
-                <mesh filename="package://mp_description/meshes/mp_link6.STL" scale= "0.01 0.01 0.01"/>
+            <origin rpy="${PI} ${PI/2} ${PI}" xyz="-0.25 0.25 0"/>
+            <geometry>
+                <cylinder radius="0.1" length="0.1"/> <!-- Adjust dimensions -->
             </geometry>
         </collision>
@@ -245,7 +244,7 @@
         </visual>
         <collision>
-            <origin rpy="${PI/2} 0 ${PI/2}" xyz="-0.2 -0.2 0.1"/>
-            <geometry>
-                <mesh filename="package://mp_description/meshes/mp_gripper.STL" scale= "0.01 0.01 0.01"/>
+            <origin rpy="${PI} ${PI/2} ${PI}" xyz="-0.2 -0.2 0.1"/>
+            <geometry>
+                <cylinder radius="0.1" length="0.1"/> <!-- Adjust dimensions -->
             </geometry>
         </collision>
@@ -267,5 +266,5 @@
             <origin rpy="${PI/2} 0 ${3*PI/2}" xyz="0.41 0.95 0"/>
             <geometry>
-                <mesh filename="package://mp_description/meshes/mp_gripperlink2.STL" scale="0.01 0.01 0.01"/>
+                <box size="0.01 0.01 0.01"/>
             </geometry>
         </collision>
@@ -289,5 +288,5 @@
             <origin rpy="${PI/2} 0 ${3*PI/2}" xyz="0.41 0.1 0"/>
             <geometry>
-                <mesh filename="package://mp_description/meshes/mp_gripperlink1.STL" scale="0.01 0.01 0.01"/>
+                <box size="0.01 0.01 0.01"/>
             </geometry>
         </collision>
@@ -299,5 +298,5 @@
         <origin rpy="0 -${PI/2} 0" xyz="0 0.11 0.5"/>
         <mimic joint="joint_8" multiplier="-1" offset="0"/> <!-- offset -->
-        <disable_collisions link1="gripper_left" link2="gripper_right" reason="Never"/>
+        <!-- <disable_collisions link1="gripper_left" link2="gripper_right" reason="Never"/> -->
         <limit lower="0.0" upper="${PI/2}" effort="${effort}" velocity="${velocity}"/>
     </joint>
@@ -307,32 +306,32 @@
     </joint>
     <link name="dummy_mimic_fix"/> -->
-    <!-- <joint name="camera_optical_joint" type="fixed">
-        <origin xyz="0 0 0" rpy="${-pi/2} 0 ${-pi/2}"/>
-        <parent link="camera_link"/>
+    <link name="rgb_camera">
+        <xacro:default_inertial mass="0.001"/>
+        <visual>
+            <origin rpy="${PI/2} ${PI} ${PI/2}" xyz="-0.12 0.1 0.1"/>
+            <geometry>
+                <mesh filename="package://mp_description/meshes/pi_camera.STL" scale="0.01 0.01 0.01"/>
+            </geometry>
+        </visual>
+        <collision>
+            <origin rpy="0 0 0" xyz="0 0 0"/>
+            <geometry>
+                <mesh filename="package://mp_description/meshes/pi_camera.STL" scale="0.01 0.01 0.01"/>
+            </geometry>
+        </collision>
+    </link>
+    <joint name ="rgb_camera_joint" type="fixed">
+        <parent link="gripper_support"/>
+        <child link = "rgb_camera"/>
+        <origin xyz="-0.4 0 0" rpy="0 -${PI/2} 0"/>
+        <!-- y - ${PI} -->
+    </joint>
+    <link name="camera_link_optical"/>
+    <joint name="camera_optical_joint" type="fixed">
+        <parent link="rgb_camera"/>
         <child link="camera_link_optical"/>
-    </joint>
-    <link name="camera_link_optical"></link>
-    <gazebo reference="camera_link">
-        <sensor name="camera" type="camera">
-            <pose> 0 0 0 0 0 0 </pose>
-            <visualize>true</visualize>
-            <update_rate>10</update_rate>
-            <camera>
-                <horizontal_fov>1.089</horizontal_fov>
-                <image>
-                    <format>R8G8B8</format>
-                    <width>640</width>
-                    <height>480</height>
-                </image>
-                <clip>
-                    <near>0.05</near>
-                    <far>8.0</far>
-                </clip>
-            </camera>
-            <plugin name="camera_controller" filename="libgazebo_ros_camera.so">
-                <frame_name>camera_link_optical</frame_name>
-            </plugin>
-        </sensor>
-    </gazebo> -->
+        <origin xyz="0 0 0" rpy="0 ${3*PI/2} ${PI}"/>
+        <!-- 0.55 0.125 -->
+    </joint>
     <xacro:default_transmission number="1"/>
     <xacro:default_transmission number="2"/>
@@ -344,48 +343,2 @@
     <xacro:default_transmission number="8"/>
 </robot>
-<!--
-<link name="gripper_right">
-        <xacro:default_inertial mass="0.01"/>
-        <visual>
-            <origin rpy="0 0 -${PI/2}" xyz="-0.1 0.5 -0.1"/>
-            <geometry>
-                <mesh filename="package://arduinobot_description/meshes/right_finger.STL" scale="0.01 0.01 0.01"/>
-            </geometry>
-        </visual>
-        <collision>
-            <origin rpy="0 0 -${PI/2}" xyz="-0.1 0.5 -0.1"/>
-            <geometry>
-                <mesh filename="package://arduinobot_description/meshes/right_finger.STL" scale="0.01 0.01 0.01"/>
-            </geometry>
-        </collision>
-    </link>
-    <link name="gripper_left">
-        <xacro:default_inertial mass="0.01"/>
-        <visual>
-            <origin rpy="0 0 -${PI/2}" xyz="-0.04 0.5 -0.1"/>
-            <geometry>
-                <mesh filename="package://arduinobot_description/meshes/left_finger.STL" scale="0.01 0.01 0.01"/>
-            </geometry>
-        </visual>
-        <collision>
-            <origin rpy="0 0 -${PI/2}" xyz="-0.04 0.5 -0.1"/>
-            <geometry>
-                <mesh filename="package://arduinobot_description/meshes/left_finger.STL" scale="0.01 0.01 0.01"/>
-            </geometry>
-        </collision>
-    </link>
-    <joint name="joint_4" type="revolute">
-        <parent link="claw_support"/>
-        <child link="gripper_right"/>
-        <axis xyz="0 0 1"/>
-        <origin rpy="0 0 0" xyz="-0.04 0.13 -0.1"/>
-        <limit lower="-${PI/2}" upper="0.0" effort="${effort}" velocity="${velocity}"/>
-    </joint>
-    <joint name="joint_5" type="revolute">
-        <parent link="claw_support"/>
-        <child link="gripper_left"/>
-        <axis xyz="0 0 1"/>
-        <origin rpy="0 0 0" xyz="-0.22 0.13 -0.1"/>
-        <mimic joint="joint_4" multiplier="-1"/>
-        <limit lower="0.0" upper="${PI/2}" effort="${effort}" velocity="${velocity}"/>
-    </joint> -->

File: src/mp_description/urdf/mp_gazebo.xacro (robot description, xacro)
@@ -8,3 +8,66 @@
         </plugin>
     </gazebo>
+    <gazebo reference="rgb_camera">
+        <sensor name="camera" type="camera">
+            <always_on>true</always_on>
+            <update_rate>15.0</update_rate>
+            <visualize>true</visualize>
+            <topic>image_raw</topic>  <!-- Remove leading slash -->
+            <camera name="camera">
+                <horizontal_fov>1.21126</horizontal_fov>
+                <image>
+                    <width>2304</width>
+                    <height>1296</height>
+                    <format>R8G8B8</format>
+                </image>
+                <clip>
+                    <near>0.1</near>
+                    <far>100.0</far>
+                </clip>
+            </camera>
+            <plugin name="camera_plugin" filename="libgazebo_ros_camera.so">
+                <ros>
+                    <namespace>mp</namespace>
+                </ros>
+                <camera_name>rgb_camera</camera_name>
+                <frame_name>camera_link_optical</frame_name>
+            </plugin>
+        </sensor>
+    </gazebo>
+    <!-- <gazebo reference="rgb_camera">
+    <sensor name="camera" type="camera">
+        <always_on>true</always_on>
+        <update_rate>30.0</update_rate>
+        <visualize>true</visualize>
+        <topic>image_raw</topic>
+        <camera name="camera">
+            <horizontal_fov>1.21126</horizontal_fov>
+            <image>
+                <width>2304</width>
+                <height>1296</height>
+                <format>R8G8B8</format>
+            </image>
+            <clip>
+                <near>0.1</near>
+                <far>100.0</far>
+            </clip>
+            <distortion>
+                <k1>0.0</k1>
+                <k2>0.0</k2>
+                <k3>0.0</k3>
+                <p1>0.0</p1>
+                <p2>0.0</p2>
+                <center>0.5 0.5</center>
+            </distortion>
+        </camera>
+        <plugin name="camera_controller" filename="libgazebo_ros_camera.so">
+            <ros>
+                <namespace>${namespace}</namespace>
+                <remapping>image_raw:=image</remapping>
+            </ros>
+            <camera_name>rgb_camera</camera_name>
+            <frame_name>camera_link_optical</frame_name>
+        </plugin>
+    </sensor>
+</gazebo> -->
 </robot>
